File: STM32TrialPcb.kicad_sch (KiCad schematic)
At the start: 31 parts, among them J1 USB_B_Micro, J2 Conn_01x15, J3 Conn_01x15, SW1 SW_Push, SW2 SW_Push, U1 TLV75533PDRV, U2 STM32F103C8T6, Y1 8M

Commit message: Improve layout, dimensions, symmetry.
Other:
- note removed: "GPIO Headers 01x15 - Male"
- note removed: "MCU Reset"
Changed lines of the file:
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@@
-		)
-	)
-	(text "GPIO Headers 01x15 - Male\n"
-		(exclude_from_sim no)
-		(at 32.258 102.87 0)
-		(effects
-			(font
-				(size 1.27 1.27)
-			)
-		)
-	)
-	(text "MCU Reset\n"
-		(exclude_from_sim no)
-		(at 24.384 57.15 0)
-		(effects
-			(font
-				(size 1.27 1.27)
-			)
 		)
 	)

Commit message: add assembly and move gerbers, update pcb
Parts:
- L1: footprint Inductor_SMD:L_0201_0603Metric -> Inductor_SMD:L_0603_1608Metric
- R2: footprint Resistor_SMD:R_0201_0603Metric -> Resistor_SMD:R_0402_1005Metric
Changed lines of the file:
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@@
 			)
 		)
-		(property "Footprint" "Inductor_SMD:L_0201_0603Metric"
+		(property "Footprint" "Inductor_SMD:L_0603_1608Metric"
 			(at 201.93 29.21 0)
 			(effects
@@
 			)
 		)
-		(property "Footprint" "Resistor_SMD:R_0201_0603Metric"
+		(property "Footprint" "Resistor_SMD:R_0402_1005Metric"
 			(at 245.872 96.52 90)
 			(effects
